File: branches/facedancer11/facedancer11.sch (EAGLE design)
At the start: 20 parts, among them CN1 HOST, CN2 VICTIM, Q1 12MHz, U1 F261X---PM64, U2 FT232RL-BASICSSOP, U3 MAX3420ELQFP32

Commit message: Facedancer11 pieces.
git-svn-id: https://svn.code.sf.net/p/goodfet/code@1181 12e2690d-a6be-4b82-a7b7-67c4a43b65c8
Parts:
- CN2: value VICTIM -> TARGET
Changed lines of the file:
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@@
 <part name="U3" library="active" deviceset="MAX3420E" device="LQFP32"/>
 <part name="Q1" library="crystal" deviceset="CRYSTAL" device="HC49UP" value="12MHz"/>
-<part name="CN2" library="adafruit" deviceset="USB" device="MINIB" value="VICTIM"/>
+<part name="CN2" library="adafruit" deviceset="USB" device="MINIB" value="TARGET"/>
 <part name="R3" library="rcl" deviceset="R-US_" device="R0603" value="33"/>
 <part name="R4" library="rcl" deviceset="R-US_" device="R0603" value="33"/>
