File: contrib/goodthopter10/goodthopter10.sch (EAGLE design)
At the start: 16 parts, among them IC1 F22X4---DA38, IC2 FT232RL-BASICSSOP, Q1 20MHz, X1 USBPCB, X3 KUSBVX-BS1N

Commit message: Created MCP2551 and USB-TYPE-B Library Parts for GoodThopter10.
git-svn-id: https://svn.code.sf.net/p/goodfet/code@1197 12e2690d-a6be-4b82-a7b7-67c4a43b65c8
Parts:
- removed X1: USBPCB, SparkFun:USBPCB
- removed X3: KUSBVX-BS1N, con-kycon:KUSBVX-BS1N
- added 292304-2: MINI-USB_4P-292304-2, USB-TYPE-B:MINI-USB_4P-292304-2
Connections:
- removed net RST: IC1.6
- new net !INT: IC1.27, U$1.!INT
- new net CAN_SHLD: CAN.5
- new net CAN_V+_OPT: CAN.9
- new net GND_OPT: CAN.6
- new net RSRVD0: CAN.1
- new net RSRVD1: CAN.4
- new net RSRVD2: CAN.8
- net GND: now also 292304-2.4; no longer X1.GND
- net N$3: now also 292304-2.3; no longer X1.D+
- net N$4: now also 292304-2.2; no longer X1.D-
- net VCC: now also U$1.!RST
- net VCC5V: now also 292304-2.1; no longer X1.VBUS
Other:
- note added: "292304-2"
- note added: "Add MCP2551"
- note added: "All NC inputs must be run to Vcc or GND"
- note added: "High Voltage: DB-9"
- note added: "High and low voltage needed:"
- note added: "Low Voltage: DNP Header"
Changed lines of the file:
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@@
 </classes>
 <parts>
-<part name="X1" library="SparkFun" deviceset="USB" device="PCB"/>
 <part name="GND3" library="supply1" deviceset="GND" device=""/>
 <part name="IC2" library="SparkFun" deviceset="FT232RL-BASIC" device="SSOP"/>
@@
 <part name="GND6" library="supply1" deviceset="GND" device=""/>
 <part name="P+1" library="supply1" deviceset="VCC" device=""/>
-<part name="X3" library="con-kycon" deviceset="KUSBVX-BS1N" device=""/>
+<part name="292304-2" library="USB-TYPE-B" deviceset="MINI-USB_4P-" device="292304-2"/>
 </parts>
 <sheets>
@@
 <text x="-43.18" y="15.24" size="1.778" layer="91">Andrew Righter</text>
 <text x="-43.18" y="12.7" size="1.778" layer="91">&lt;andrew.righter at gmail.com&gt;</text>
-<text x="-53.34" y="129.54" size="1.27" layer="95">Crystal - Parallel Cut Crystal</text>
-<text x="-53.34" y="132.08" size="1.27" layer="95">Notes:</text>
-<text x="-53.34" y="127" size="1.27" layer="95">No SPI operations until Osc Startup Timer (OST) Expires</text>
-<text x="-53.34" y="124.46" size="1.27" layer="95">Series resistor may be required for AT strip cut crystals (direclty out of OSC2)</text>
+<text x="101.6" y="147.32" size="1.27" layer="95">Crystal - Parallel Cut Crystal</text>
+<text x="101.6" y="149.86" size="1.27" layer="95">Notes:</text>
+<text x="101.6" y="144.78" size="1.27" layer="95">No SPI operations until Osc Startup Timer (OST) Expires</text>
+<text x="101.6" y="142.24" size="1.27" layer="95">Series resistor may be required for AT strip cut crystals (direclty out of OSC2)</text>
 <text x="-40.64" y="91.44" size="1.27" layer="95">MCP2515 Crystal Circuit</text>
+<text x="-40.64" y="60.96" size="1.778" layer="95" rot="R90">292304-2</text>
+<text x="101.6" y="139.7" size="1.27" layer="95">All NC inputs must be run to Vcc or GND</text>
+<text x="101.6" y="134.62" size="1.778" layer="91">High and low voltage needed:</text>
+<text x="104.14" y="132.08" size="1.778" layer="91">High Voltage: DB-9</text>
+<text x="104.14" y="129.54" size="1.778" layer="91">Low Voltage: DNP Header</text>
+<text x="101.6" y="127" size="1.778" layer="91">Add MCP2551</text>
 </plain>
 <instances>
-<instance part="X1" gate="G$1" x="-22.86" y="71.12" rot="R180"/>
 <instance part="GND3" gate="1" x="-20.32" y="78.74" rot="R180"/>
 <instance part="IC2" gate="G$1" x="12.7" y="53.34"/>
@@
 <instance part="CAN" gate="G$1" x="121.92" y="99.06"/>
 <instance part="Q1" gate="G$1" x="-22.86" y="104.14" rot="R90"/>
-<instance part="GND2" gate="1" x="106.68" y="93.98"/>
+<instance part="GND2" gate="1" x="99.06" y="93.98"/>
 <instance part="GND6" gate="1" x="30.48" y="86.36"/>
 <instance part="P+1" gate="VCC" x="83.82" y="119.38"/>
-<instance part="X3" gate="G$1" x="-45.72" y="68.58" rot="R180"/>
+<instance part="292304-2" gate="G$1" x="-33.02" y="68.58" rot="R180"/>
 </instances>
 <busses>
@@
 <pinref part="P+1" gate="VCC" pin="VCC"/>
 <wire x1="83.82" y1="114.3" x2="83.82" y2="116.84" width="0.1524" layer="91"/>
+<pinref part="U$1" gate="G$1" pin="!RST"/>
+<wire x1="76.2" y1="111.76" x2="83.82" y2="111.76" width="0.1524" layer="91"/>
+<wire x1="83.82" y1="111.76" x2="83.82" y2="114.3" width="0.1524" layer="91"/>
+<junction x="83.82" y="114.3"/>
 </segment>
 </net>
@@
 <net name="GND" class="0">
 <segment>
+<pinref part="GND3" gate="1" pin="GND"/>
+<wire x1="-27.94" y1="71.12" x2="-20.32" y2="71.12" width="0.1524" layer="91"/>
 <wire x1="-20.32" y1="71.12" x2="-20.32" y2="76.2" width="0.1524" layer="91"/>
-<pinref part="X1" gate="G$1" pin="GND"/>
-<pinref part="GND3" gate="1" pin="GND"/>
+<pinref part="292304-2" gate="G$1" pin="4"/>
 </segment>
 <segment>
@@
 <segment>
 <pinref part="CAN" gate="G$1" pin="3"/>
-<wire x1="114.3" y1="99.06" x2="106.68" y2="99.06" width="0.1524" layer="91"/>
+<wire x1="114.3" y1="99.06" x2="99.06" y2="99.06" width="0.1524" layer="91"/>
 <pinref part="GND2" gate="1" pin="GND"/>
-<wire x1="106.68" y1="99.06" x2="106.68" y2="96.52" width="0.1524" layer="91"/>
+<wire x1="99.06" y1="99.06" x2="99.06" y2="96.52" width="0.1524" layer="91"/>
 </segment>
 <segment>
@@
 <segment>
 <wire x1="-20.32" y1="63.5" x2="-2.54" y2="63.5" width="0.1524" layer="91"/>
-<pinref part="X1" gate="G$1" pin="D+"/>
 <pinref part="IC2" gate="G$1" pin="USBDP"/>
+<wire x1="-20.32" y1="63.5" x2="-20.32" y2="68.58" width="0.1524" layer="91"/>
+<wire x1="-20.32" y1="68.58" x2="-27.94" y2="68.58" width="0.1524" layer="91"/>
+<pinref part="292304-2" gate="G$1" pin="3"/>
 </segment>
 </net>
 <net name="N$4" class="0">
 <segment>
-<wire x1="-2.54" y1="66.04" x2="-20.32" y2="66.04" width="0.1524" layer="91"/>
+<wire x1="-2.54" y1="66.04" x2="-27.94" y2="66.04" width="0.1524" layer="91"/>
 <pinref part="IC2" gate="G$1" pin="USBDM"/>
-<pinref part="X1" gate="G$1" pin="D-"/>
+<pinref part="292304-2" gate="G$1" pin="2"/>
 </segment>
 </net>
@@
 </segment>
 </net>
-<net name="RST" class="0">
-<segment>
-<wire x1="78.74" y1="58.42" x2="71.12" y2="58.42" width="0.1524" layer="91"/>
-<label x="71.12" y="58.42" size="1.778" layer="95"/>
-<pinref part="IC1" gate="G$1" pin="6"/>
-</segment>
-</net>
 <net name="RTS" class="0">
 <segment>
@@
 <net name="VCC5V" class="0">
 <segment>
-<wire x1="-20.32" y1="68.58" x2="-7.62" y2="68.58" width="0.1524" layer="91"/>
-<wire x1="-7.62" y1="68.58" x2="-7.62" y2="58.42" width="0.1524" layer="91"/>
-<wire x1="-7.62" y1="58.42" x2="-2.54" y2="58.42" width="0.1524" layer="91"/>
-<label x="-17.78" y="68.58" size="1.778" layer="95"/>
-<pinref part="X1" gate="G$1" pin="VBUS"/>
+<wire x1="-22.86" y1="58.42" x2="-2.54" y2="58.42" width="0.1524" layer="91"/>
+<label x="-22.86" y="58.42" size="1.778" layer="95"/>
 <pinref part="IC2" gate="G$1" pin="VCC"/>
+<wire x1="-27.94" y1="63.5" x2="-22.86" y2="63.5" width="0.1524" layer="91"/>
+<wire x1="-22.86" y1="63.5" x2="-22.86" y2="58.42" width="0.1524" layer="91"/>
+<pinref part="292304-2" gate="G$1" pin="1"/>
 </segment>
 </net>
@@
 <pinref part="CAN" gate="G$1" pin="7"/>
 <wire x1="129.54" y1="99.06" x2="137.16" y2="99.06" width="0.1524" layer="91"/>
-<label x="129.54" y="99.06" size="1.778" layer="95"/>
+<label x="129.54" y="99.06" size="1.27" layer="95"/>
 </segment>
 </net>
@@
 <segment>
 <pinref part="CAN" gate="G$1" pin="2"/>
-<wire x1="114.3" y1="101.6" x2="106.68" y2="101.6" width="0.1524" layer="91"/>
-<label x="106.68" y="101.6" size="1.778" layer="95"/>
-</segment>
-</net>
+<wire x1="114.3" y1="101.6" x2="104.14" y2="101.6" width="0.1524" layer="91"/>
+<label x="104.14" y="101.6" size="1.27" layer="95"/>
+</segment>
+</net>
+<net name="!INT" class="0">
+<segment>
+<pinref part="U$1" gate="G$1" pin="!INT"/>
+<wire x1="76.2" y1="96.52" x2="83.82" y2="96.52" width="0.1524" layer="91"/>
+<label x="78.74" y="96.52" size="1.778" layer="95"/>
+</segment>
+<segment>
+<pinref part="IC1" gate="G$1" pin="27"/>
+<wire x1="147.32" y1="43.18" x2="154.94" y2="43.18" width="0.1524" layer="91"/>
+<label x="149.86" y="43.18" size="1.778" layer="95"/>
+</segment>
+</net>
+<net name="GND_OPT" class="0">
+<segment>
+<pinref part="CAN" gate="G$1" pin="6"/>
+<wire x1="129.54" y1="101.6" x2="137.16" y2="101.6" width="0.1524" layer="91"/>
+<label x="129.54" y="101.6" size="1.27" layer="95"/>
+</segment>
+</net>
+<net name="RSRVD2" class="0">
+<segment>
+<pinref part="CAN" gate="G$1" pin="8"/>
+<wire x1="129.54" y1="96.52" x2="137.16" y2="96.52" width="0.1524" layer="91"/>
+<label x="129.54" y="96.52" size="1.27" layer="95"/>
+</segment>
+</net>
+<net name="CAN_V+_OPT" class="0">
+<segment>
+<pinref part="CAN" gate="G$1" pin="9"/>
+<wire x1="129.54" y1="93.98" x2="137.16" y2="93.98" width="0.1524" layer="91"/>
+<label x="129.54" y="93.98" size="1.27" layer="95"/>
+</segment>
+</net>
+<net name="CAN_SHLD" class="0">
+<segment>
+<pinref part="CAN" gate="G$1" pin="5"/>
+<wire x1="114.3" y1="93.98" x2="104.14" y2="93.98" width="0.1524" layer="91"/>
+<label x="104.14" y="93.98" size="1.27" layer="95"/>
+</segment>
+</net>
+<net name="RSRVD1" class="0">
+<segment>
+<pinref part="CAN" gate="G$1" pin="4"/>
+<wire x1="114.3" y1="96.52" x2="104.14" y2="96.52" width="0.1524" layer="91"/>
+<label x="104.14" y="96.52" size="1.27" layer="95"/>
+</segment>
+</net>
+<net name="RSRVD0" class="0">
+<segment>
+<pinref part="CAN" gate="G$1" pin="1"/>
+<wire x1="114.3" y1="104.14" x2="104.14" y2="104.14" width="0.1524" layer="91"/>
+<label x="104.14" y="104.14" size="1.27" layer="95"/>
+</segment>
+</net>

Commit message: Updated schematic /goodthopter10, added CAN_IO, MCP2551 and Low/High Voltage options.
git-svn-id: https://svn.code.sf.net/p/goodfet/code@1199 12e2690d-a6be-4b82-a7b7-67c4a43b65c8
Parts:
- added C5, C6: 0.1uF, rcl:C-EUC0603
- added CAN_IO: (no value), con-lstb:MA06-1
- added R2, R3: 470, rcl:R-US_R0603
- added R4: 10k, rcl:R-US_R0603
- added RX_LED, TX_LED: (no value), led:LEDCHIP-LED0603
- added U$2: MCP2551, MCP2551:MCP2551
- renumbered CAN to CAN(12V)
Connections:
- new net !TX0RTS: CAN_IO.4, U$1.!TX0RTS
- new net !TX1RTS: CAN_IO.5, U$1.!TX1RTS
- new net !TX2RTS: CAN_IO.6, U$1.!TX2RTS
- new net CANH: CAN(12V).7, U$2.CANH
- new net CANL: CAN(12V).2, U$2.CANL
- new net CLKOUT: CAN_IO.3, U$1.CLKOUT/SOF
- new net N$1: R2.2, RX_LED.A
- new net N$11: C6.2, R4.1
- new net N$2: R3.2, TX_LED.A
- new net N$5: R4.2, U$1.!RST
- net !CS: no longer U$1.!CS
- net GND: now also C5.1, C6.1, U$2.RS, U$2.VSS
- net RXCAN: now also CAN_IO.2, RX_LED.C, U$2.RXD; no longer CAN(12V).2
- net TXCAN: now also CAN_IO.1, TX_LED.C, U$2.TXD; no longer CAN(12V).7
- net VCC: now also R2.1, R3.1; no longer U$1.!RST
- net VCC5V: now also C5.2, U$2.VDD
Other:
- note removed: "Add MCP2551"
- note removed: "High Voltage: DB-9"
- note removed: "High and low voltage needed:"
- note removed: "Low Voltage: DNP Header"
- moved on the sheet: R10

Commit message: Added BOM to GoodThopter10/, modified SCH and BRD.
git-svn-id: https://svn.code.sf.net/p/goodfet/code@1212 12e2690d-a6be-4b82-a7b7-67c4a43b65c8
Parts:
- removed Q1: 20MHz, crystal:CRYSTALMM20SS
- added Q2: 20MHz, crystal:CRYSTALHC49UP
- R10: value 300 -> 330
Connections:
- removed net !CS: IC1.11
- net OSC1: now also Q2.1; no longer Q1.1
- net OSC2: now also Q2.2; no longer Q1.2
- net VCC: now also C5.2, U$2.VDD
- net VCC5V: no longer C5.2, U$2.VDD
Changed lines of the file:
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@@
 <part name="TXLED" library="led" deviceset="LED" device="CHIP-LED0603"/>
 <part name="P+4" library="supply1" deviceset="VCC" device=""/>
-<part name="R10" library="rcl" deviceset="R-US_" device="R0603" value="300"/>
+<part name="R10" library="rcl" deviceset="R-US_" device="R0603" value="330"/>
 <part name="C4" library="rcl" deviceset="C-EU" device="C0603" value="0.1µF"/>
 <part name="P+5" library="supply1" deviceset="VCC" device=""/>
@@
 <part name="GND1" library="supply1" deviceset="GND" device=""/>
 <part name="CAN(12V)" library="SparkFun-Connectors" deviceset="DB9" device="MALE"/>
-<part name="Q1" library="crystal" deviceset="CRYSTAL" device="MM20SS" value="20MHz"/>
 <part name="GND2" library="supply1" deviceset="GND" device=""/>
 <part name="GND6" library="supply1" deviceset="GND" device=""/>
@@
 <part name="GND7" library="supply1" deviceset="GND" device=""/>
 <part name="GND9" library="supply1" deviceset="GND" device=""/>
-<part name="P+2" library="supply1" deviceset="VCC" device=""/>
 <part name="C5" library="rcl" deviceset="C-EU" device="C0603" value="0.1uF"/>
 <part name="GND10" library="supply1" deviceset="GND" device=""/>
@@
 <part name="P+1" library="supply1" deviceset="VCC" device=""/>
 <part name="CAN_IO" library="con-lstb" deviceset="MA06-1" device=""/>
+<part name="VCC5V" library="supply1" deviceset="VCC" device=""/>
+<part name="Q2" library="crystal" deviceset="CRYSTAL" device="HC49UP" value="20MHz"/>
 </parts>
 <sheets>
@@
 <instance part="GND1" gate="1" x="-48.26" y="96.52"/>
 <instance part="CAN(12V)" gate="G$1" x="121.92" y="99.06"/>
-<instance part="Q1" gate="G$1" x="-22.86" y="104.14" rot="R90"/>
 <instance part="GND2" gate="1" x="99.06" y="93.98"/>
 <instance part="GND6" gate="1" x="35.56" y="81.28"/>
@@
 <instance part="GND7" gate="1" x="20.32" y="147.32" rot="R180"/>
 <instance part="GND9" gate="1" x="-35.56" y="132.08"/>
-<instance part="P+2" gate="VCC" x="-30.48" y="167.64"/>
 <instance part="C5" gate="G$1" x="-22.86" y="154.94" rot="R180"/>
 <instance part="GND10" gate="1" x="-22.86" y="149.86"/>
@@
 <instance part="P+1" gate="VCC" x="81.28" y="139.7"/>
 <instance part="CAN_IO" gate="1" x="68.58" y="149.86" rot="R180"/>
+<instance part="VCC5V" gate="VCC" x="-30.48" y="170.18"/>
+<instance part="Q2" gate="G$1" x="-22.86" y="104.14" rot="R90"/>
 </instances>
 <busses>
 </busses>
 <nets>
-<net name="!CS" class="0">
-<segment>
-<wire x1="78.74" y1="45.72" x2="71.12" y2="45.72" width="0.1524" layer="91"/>
-<label x="71.12" y="45.72" size="1.778" layer="95"/>
-<pinref part="IC1" gate="G$1" pin="11"/>
-</segment>
-</net>
 <net name="MOSI" class="0">
 <segment>
@@
 <wire x1="81.28" y1="109.22" x2="81.28" y2="137.16" width="0.1524" layer="91"/>
 <pinref part="P+1" gate="VCC" pin="VCC"/>
+</segment>
+<segment>
+<pinref part="U$2" gate="G$1" pin="VDD"/>
+<wire x1="-20.32" y1="134.62" x2="-30.48" y2="134.62" width="0.1524" layer="91"/>
+<wire x1="-30.48" y1="134.62" x2="-30.48" y2="162.56" width="0.1524" layer="91"/>
+<wire x1="-30.48" y1="162.56" x2="-30.48" y2="165.1" width="0.1524" layer="91"/>
+<wire x1="-30.48" y1="162.56" x2="-22.86" y2="162.56" width="0.1524" layer="91"/>
+<wire x1="-22.86" y1="162.56" x2="-22.86" y2="160.02" width="0.1524" layer="91"/>
+<junction x="-30.48" y="162.56"/>
+<pinref part="C5" gate="G$1" pin="2"/>
+<label x="-30.48" y="144.78" size="1.778" layer="95" rot="R90"/>
+<pinref part="VCC5V" gate="VCC" pin="VCC"/>
+<wire x1="-30.48" y1="167.64" x2="-30.48" y2="162.56" width="0.1524" layer="91"/>
 </segment>
 </net>
@@
 <pinref part="292304-2" gate="G$1" pin="1"/>
 </segment>
-<segment>
-<pinref part="U$2" gate="G$1" pin="VDD"/>
-<wire x1="-20.32" y1="134.62" x2="-30.48" y2="134.62" width="0.1524" layer="91"/>
-<wire x1="-30.48" y1="134.62" x2="-30.48" y2="162.56" width="0.1524" layer="91"/>
-<pinref part="P+2" gate="VCC" pin="VCC"/>
-<wire x1="-30.48" y1="162.56" x2="-30.48" y2="165.1" width="0.1524" layer="91"/>
-<wire x1="-30.48" y1="162.56" x2="-22.86" y2="162.56" width="0.1524" layer="91"/>
-<wire x1="-22.86" y1="162.56" x2="-22.86" y2="160.02" width="0.1524" layer="91"/>
-<junction x="-30.48" y="162.56"/>
-<pinref part="C5" gate="G$1" pin="2"/>
-<label x="-30.48" y="144.78" size="1.778" layer="95" rot="R90"/>
-</segment>
 </net>
 <net name="OSC1" class="0">
@@
 <wire x1="-22.86" y1="99.06" x2="-22.86" y2="93.98" width="0.1524" layer="91"/>
 <label x="-22.86" y="93.98" size="1.778" layer="95"/>
-<pinref part="Q1" gate="G$1" pin="1"/>
 <wire x1="-22.86" y1="101.6" x2="-22.86" y2="99.06" width="0.1524" layer="91"/>
 <junction x="-22.86" y="99.06"/>
+<pinref part="Q2" gate="G$1" pin="1"/>
 </segment>
 <segment>
@@
 <wire x1="-22.86" y1="111.76" x2="-22.86" y2="116.84" width="0.1524" layer="91"/>
 <label x="-22.86" y="116.84" size="1.778" layer="95"/>
-<pinref part="Q1" gate="G$1" pin="2"/>
 <wire x1="-22.86" y1="106.68" x2="-22.86" y2="111.76" width="0.1524" layer="91"/>
 <junction x="-22.86" y="111.76"/>
-</segment>
-<segment>
+<pinref part="Q2" gate="G$1" pin="2"/>
+</segment>
+<segment>

Commit message: Updated Routing/SCH and Produced Gerbers
git-svn-id: https://svn.code.sf.net/p/goodfet/code@1216 12e2690d-a6be-4b82-a7b7-67c4a43b65c8
Parts:
- R2, R3: value 470 -> 330
Connections:
- net N$3 renamed USBDP
- net N$4 renamed USBDM
- removed net N$11: C6.2, R4.1
- new net !CS: IC1.11, U$1.!CS
- net VCC: now also C6.2, R4.1
Other:
- note added: "Test Only: Do Not Populate"
- note removed: "<Travis at RadiantMachines.com>"
- note removed: "Travis Goodspeed"
