File: branches/facedancer20/facedancer20.brd (EAGLE design)
At the start: 71.1 x 23.5 mm, 20 parts, among them CN1 HOST, CN2 TARGET, CN3 USB-A-S, Q1 12MHz, U1 F261X---PM64, U2 FT232RL-BASICSSOP, U4 MAX3421ESMD

Commit message: FD20 ready for first test run.
git-svn-id: https://svn.code.sf.net/p/goodfet/code@1346 12e2690d-a6be-4b82-a7b7-67c4a43b65c8
Connections:
- removed net N$9: U4.17
- new net GPX: U1.43, U4.17
Routing:
- net GPX: track 0.00 -> 9.06 mm
- net GND: track 43.8 -> 45.3 mm
Changed lines of the file:
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@@
 </element>
 <element name="U2" library="SparkFun" package="SSOP28DB" value="FT232RL-BASICSSOP" x="16.51" y="9.8425" smashed="yes" rot="R180">
-<attribute name="NAME" x="13.97" y="12.065" size="0.8128" layer="25" rot="R180"/>
+<attribute name="NAME" x="13.57" y="15.465" size="0.8128" layer="25" rot="R180"/>
 <attribute name="VALUE" x="20.955" y="9.8425" size="0.4064" layer="27" rot="R180"/>
 </element>
@@
 <element name="C7" library="rcl" package="C0603" value="18pF" x="44.2" y="7.6" smashed="yes">
 <attribute name="NAME" x="43.565" y="8.235" size="0.4064" layer="25" font="vector"/>
-<attribute name="VALUE" x="43.565" y="8.695" size="0.4064" layer="27" font="fixed"/>
 </element>
 <element name="U4" library="SparkFun-DigitalIC" package="TQFP32-5MM" value="MAX3421ESMD" x="47.4" y="14.6" smashed="yes" rot="R270">
@@
 <contactref element="C2" pad="1"/>
 <contactref element="CN1" pad="GND"/>
-<wire x1="19.435" y1="6.1865" x2="18.785" y2="6.1865" width="0.254" layer="1"/>
-<wire x1="19.435" y1="6.1865" x2="19.435" y2="8.3225" width="0.254" layer="1"/>
+<wire x1="19.435" y1="6.1865" x2="19.435" y2="8" width="0.254" layer="1"/>
+<wire x1="19.435" y1="8" x2="19.435" y2="8.3225" width="0.254" layer="1"/>
 <wire x1="19.435" y1="8.3225" x2="19.685" y2="8.5725" width="0.254" layer="1"/>
 <wire x1="19.685" y1="8.5725" x2="23.28" y2="8.5725" width="0.254" layer="1"/>
@@
 <wire x1="16.185" y1="6.1865" x2="16.185" y2="11.105" width="0.254" layer="1"/>
 <wire x1="16.185" y1="11.105" x2="16.8275" y2="11.7475" width="0.254" layer="1"/>
-<wire x1="19.435" y1="4.6275" x2="19.435" y2="6.1865" width="0.254" layer="1"/>
-<wire x1="19.3675" y1="3.2425" x2="19.435" y2="4.6275" width="0.254" layer="1"/>
 <wire x1="29.3175" y1="16.085" x2="29.3175" y2="14.3725" width="0.254" layer="1"/>
 <wire x1="29.7425" y1="16.51" x2="29.3175" y2="16.085" width="0.254" layer="1"/>
@@
 <wire x1="44.8" y1="21.6" x2="45" y2="21.6" width="0.254" layer="16"/>
 <wire x1="45" y1="21.6" x2="45" y2="21.4" width="0.254" layer="16"/>
+<wire x1="19.435" y1="6.1865" x2="19.435" y2="3.31" width="0.254" layer="1"/>
+<wire x1="19.435" y1="3.31" x2="19.3675" y2="3.2425" width="0.254" layer="1"/>
+<wire x1="18.785" y1="6.1865" x2="18.785" y2="7.35" width="0.254" layer="1"/>
+<wire x1="18.785" y1="7.35" x2="19.435" y2="8" width="0.254" layer="1"/>
 </signal>
 <signal name="N$1">
 <contactref element="R1" pad="2"/>
 <contactref element="U1" pad="12"/>
-<wire x1="22.7875" y1="6.8225" x2="26.2675" y2="6.8225" width="0.254" layer="1"/>
-<wire x1="22.86" y1="3.3425" x2="22.7875" y2="6.8225" width="0.254" layer="1"/>
+<wire x1="26.2675" y1="6.8225" x2="22.86" y2="6.8225" width="0.254" layer="1"/>
+<wire x1="22.86" y1="6.8225" x2="22.86" y2="3.3425" width="0.254" layer="1"/>
 </signal>
 <signal name="N$2">
@@
 <contactref element="U2" pad="22"/>
 <contactref element="RXLED" pad="C"/>
-<wire x1="16.835" y1="4.885" x2="16.835" y2="6.1865" width="0.254" layer="1"/>
-<wire x1="15.9925" y1="3.2425" x2="16.835" y2="4.885" width="0.254" layer="1"/>
+<wire x1="16.835" y1="6.1865" x2="16.835" y2="4.085" width="0.254" layer="1"/>
+<wire x1="16.835" y1="4.085" x2="15.9925" y2="3.2425" width="0.254" layer="1"/>
 </signal>
 <signal name="N$7">
 <contactref element="U2" pad="23"/>
 <contactref element="TXLED" pad="C"/>
-<wire x1="17.485" y1="4.5375" x2="17.485" y2="6.1865" width="0.254" layer="1"/>
-<wire x1="17.485" y1="4.5375" x2="17.78" y2="3.2425" width="0.254" layer="1"/>
+<wire x1="17.485" y1="6.1865" x2="17.485" y2="3.5375" width="0.254" layer="1"/>
+<wire x1="17.485" y1="3.5375" x2="17.78" y2="3.2425" width="0.254" layer="1"/>
 </signal>
 <signal name="N$8">
@@
 <wire x1="54.7575" y1="8.2425" x2="61.4425" y2="8.2425" width="0.254" layer="1"/>
 </signal>
-<signal name="N$9">
+<signal name="GPX">
 <contactref element="U4" pad="17"/>
+<contactref element="U1" pad="43"/>
+<wire x1="37.8675" y1="9.8225" x2="45.65" y2="9.8225" width="0.254" layer="1"/>
+<wire x1="45.65" y1="9.8225" x2="45.65" y2="11.1" width="0.254" layer="1"/>
 </signal>
 <signal name="D-">
@@
 </signal>
 </signals>
+<errors>
+</errors>
 </board>
 </drawing>
