File: branches/goodthopter12/goodthopter12.sch (EAGLE design)
At the start: 28 parts, among them IC1 F22X4---DA38, IC2 FT232RL-BASICSSOP, Q2 20MHz

Commit message: GoodThopter12 mods.  Geting closer to manufacturing.
git-svn-id: https://svn.code.sf.net/p/goodfet/code@1565 12e2690d-a6be-4b82-a7b7-67c4a43b65c8
Parts:
- removed CAN_IO: (no value), con-lstb:MA06-1
Connections:
- removed net CAN_V+_OPT: CAN(12V).9
- removed net GND_OPT: CAN(12V).6
- removed net RSRVD0: CAN(12V).1
- removed net RSRVD1: CAN(12V).4
- removed net RSRVD2: CAN(12V).8
- new net N$11: CAN(12V).5, R5.2
- new net N$12: CAN(12V).7, R6.1
- new net N$3: CAN(12V).2, R8.2
- new net N$4: CAN(12V).3, R7.2
- net !TX0RTS: no longer CAN_IO.4
- net !TX1RTS: no longer CAN_IO.5
- net !TX2RTS: no longer CAN_IO.6
- net CANH: now also R6.2; no longer CAN(12V).3, CAN(12V).7, R5.1, R5.2, R7.2
- net CANL: now also R5.1; no longer CAN(12V).2, CAN(12V).5, R6.1, R6.2, R8.2
- net CLKOUT: no longer CAN_IO.3
- net RXCAN: no longer CAN_IO.2
- net TXCAN: no longer CAN_IO.1
Other:
- note added: "Different CAN cables need different pins."
- note added: "Known cables:"
- note added: "PAY ATTENTION!"
- note added: "Populate *TWO* of R5, R6, R7, and R8 to choose your cable."
- note added: "R5,R7 -- Pins 3,5 -- Sparkfun"
- note added: "R6,R8 -- Pins 7,2 -- Intrepid Control Systems"
- note removed: "Test Only: Do Not Populate"
- moved on the sheet: R5, R6, R7, R8
Changed lines of the file:
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@@
 <?xml version="1.0" encoding="utf-8"?>
 <!DOCTYPE eagle SYSTEM "eagle.dtd">
-<eagle version="6.2">
+<eagle version="6.3">
 <drawing>
 <settings>
@@
 <part name="GND11" library="supply1" deviceset="GND" device=""/>
 <part name="P+1" library="supply1" deviceset="VCC" device=""/>
-<part name="CAN_IO" library="con-lstb" deviceset="MA06-1" device=""/>
 <part name="Q2" library="crystal" deviceset="CRYSTAL" device="HC49UP" value="20MHz"/>
 <part name="U$2" library="MCP2551" deviceset="MCP2551" device=""/>
+<part name="R7" library="rcl" deviceset="R-US_" device="R0603" value="0"/>
+<part name="R8" library="rcl" deviceset="R-US_" device="R0603" value="0"/>
 <part name="R5" library="rcl" deviceset="R-US_" device="R0603" value="0"/>
 <part name="R6" library="rcl" deviceset="R-US_" device="R0603" value="0"/>
-<part name="R7" library="rcl" deviceset="R-US_" device="R0603" value="0"/>
-<part name="R8" library="rcl" deviceset="R-US_" device="R0603" value="0"/>
 </parts>
 <sheets>
@@
 <text x="-40.64" y="60.96" size="1.778" layer="95" rot="R90">292304-2</text>
 <text x="101.6" y="139.7" size="1.27" layer="95">All NC inputs must be run to Vcc or GND</text>
-<text x="45.72" y="162.56" size="1.778" layer="91">Test Only: Do Not Populate</text>
 <text x="-17.78" y="0" size="1.778" layer="91">Ryan Barnes</text>
+<text x="101.6" y="132.08" size="1.778" layer="104">PAY ATTENTION!</text>
+<text x="101.6" y="129.54" size="1.778" layer="104">Different CAN cables need different pins.</text>
+<text x="101.6" y="127" size="1.778" layer="104">Populate *TWO* of R5, R6, R7, and R8 to choose your cable.</text>
+<text x="101.6" y="124.46" size="1.778" layer="104">Known cables:</text>
+<text x="104.14" y="121.92" size="1.778" layer="104">R5,R7 -- Pins 3,5 -- Sparkfun</text>
+<text x="104.14" y="119.38" size="1.778" layer="104">R6,R8 -- Pins 7,2 -- Intrepid Control Systems</text>
 </plain>
 <instances>
@@
 <instance part="GND11" gate="1" x="76.2" y="119.38"/>
 <instance part="P+1" gate="VCC" x="81.28" y="139.7"/>
-<instance part="CAN_IO" gate="1" x="68.58" y="149.86" rot="R180"/>
 <instance part="Q2" gate="G$1" x="-22.86" y="104.14" rot="R90"/>
 <instance part="U$2" gate="G$1" x="-5.08" y="137.16"/>
-<instance part="R5" gate="G$1" x="27.94" y="137.16"/>
-<instance part="R6" gate="G$1" x="38.1" y="134.62"/>
-<instance part="R7" gate="G$1" x="114.3" y="104.14"/>
-<instance part="R8" gate="G$1" x="114.3" y="106.68"/>
+<instance part="R7" gate="G$1" x="124.46" y="104.14"/>
+<instance part="R8" gate="G$1" x="116.84" y="106.68"/>
+<instance part="R5" gate="G$1" x="116.84" y="99.06"/>
+<instance part="R6" gate="G$1" x="152.4" y="104.14"/>
 </instances>
 <busses>
@@
 <pinref part="U$2" gate="G$1" pin="TXD"/>
 </segment>
-<segment>
-<pinref part="CAN_IO" gate="1" pin="1"/>
-<wire x1="60.96" y1="157.48" x2="50.8" y2="157.48" width="0.1524" layer="91"/>
-<label x="50.8" y="157.48" size="1.778" layer="95"/>
-</segment>
 </net>
 <net name="RXCAN" class="0">
@@
 <pinref part="U$2" gate="G$1" pin="RXD"/>
 </segment>
-<segment>
-<pinref part="CAN_IO" gate="1" pin="2"/>
-<wire x1="60.96" y1="154.94" x2="50.8" y2="154.94" width="0.1524" layer="91"/>
-<label x="50.8" y="154.94" size="1.778" layer="95"/>
-</segment>
 </net>
 <net name="!INT" class="0">
@@
 </segment>
 </net>
-<net name="GND_OPT" class="0">
-<segment>
-<pinref part="CAN(12V)" gate="G$1" pin="6"/>
-<wire x1="144.78" y1="106.68" x2="152.4" y2="106.68" width="0.1524" layer="91"/>
-<label x="144.78" y="106.68" size="1.27" layer="95"/>
-</segment>
-</net>
-<net name="RSRVD2" class="0">
-<segment>
-<pinref part="CAN(12V)" gate="G$1" pin="8"/>
-<wire x1="144.78" y1="101.6" x2="152.4" y2="101.6" width="0.1524" layer="91"/>
-<label x="144.78" y="101.6" size="1.27" layer="95"/>
-</segment>
-</net>
-<net name="CAN_V+_OPT" class="0">
-<segment>
-<pinref part="CAN(12V)" gate="G$1" pin="9"/>
-<wire x1="144.78" y1="99.06" x2="152.4" y2="99.06" width="0.1524" layer="91"/>
-<label x="144.78" y="99.06" size="1.27" layer="95"/>
-</segment>
-</net>
-<net name="RSRVD1" class="0">
-<segment>
-<pinref part="CAN(12V)" gate="G$1" pin="4"/>
-<wire x1="129.54" y1="101.6" x2="119.38" y2="101.6" width="0.1524" layer="91"/>
-<label x="119.38" y="101.6" size="1.27" layer="95"/>
-</segment>
-</net>
-<net name="RSRVD0" class="0">
-<segment>
-<pinref part="CAN(12V)" gate="G$1" pin="1"/>
-<wire x1="129.54" y1="109.22" x2="119.38" y2="109.22" width="0.1524" layer="91"/>
-<label x="119.38" y="109.22" size="1.27" layer="95"/>
-</segment>
-</net>
 <net name="CANL" class="0">
 <segment>
-<wire x1="12.7" y1="134.62" x2="33.02" y2="134.62" width="0.1524" layer="91"/>
+<wire x1="12.7" y1="134.62" x2="20.32" y2="134.62" width="0.1524" layer="91"/>
 <label x="12.7" y="134.62" size="1.778" layer="95"/>
 <pinref part="U$2" gate="G$1" pin="CANL"/>
-<pinref part="R6" gate="G$1" pin="1"/>
-</segment>
-<segment>
-<pinref part="CAN(12V)" gate="G$1" pin="2"/>
-<wire x1="129.54" y1="106.68" x2="119.38" y2="106.68" width="0.1524" layer="91"/>
-<label x="119.38" y="106.68" size="1.27" layer="95"/>
-<pinref part="R8" gate="G$1" pin="2"/>
-</segment>
-<segment>
-<pinref part="CAN(12V)" gate="G$1" pin="5"/>
-<wire x1="129.54" y1="99.06" x2="119.38" y2="99.06" width="0.1524" layer="91"/>
-<label x="119.38" y="99.06" size="1.27" layer="95"/>
-</segment>
-<segment>
-<pinref part="R6" gate="G$1" pin="2"/>
-<wire x1="43.18" y1="134.62" x2="45.72" y2="134.62" width="0.1524" layer="91"/>
 </segment>
 <segment>
 <pinref part="R8" gate="G$1" pin="1"/>
-<wire x1="109.22" y1="106.68" x2="104.14" y2="106.68" width="0.1524" layer="91"/>
+<wire x1="111.76" y1="106.68" x2="104.14" y2="106.68" width="0.1524" layer="91"/>
+<label x="104.14" y="106.68" size="1.778" layer="95"/>
+</segment>
+<segment>
+<pinref part="R5" gate="G$1" pin="1"/>
+<wire x1="111.76" y1="99.06" x2="104.14" y2="99.06" width="0.1524" layer="91"/>
+<label x="104.14" y="99.06" size="1.778" layer="95"/>
 </segment>
 </net>
 <net name="CANH" class="0">
 <segment>
-<wire x1="12.7" y1="137.16" x2="22.86" y2="137.16" width="0.1524" layer="91"/>
+<wire x1="12.7" y1="137.16" x2="20.32" y2="137.16" width="0.1524" layer="91"/>
 <label x="12.7" y="137.16" size="1.778" layer="95"/>
 <pinref part="U$2" gate="G$1" pin="CANH"/>
-<pinref part="R5" gate="G$1" pin="1"/>
-</segment>
-<segment>
-<pinref part="CAN(12V)" gate="G$1" pin="7"/>
-<wire x1="144.78" y1="104.14" x2="152.4" y2="104.14" width="0.1524" layer="91"/>
-<label x="144.78" y="104.14" size="1.27" layer="95"/>
-</segment>
-<segment>
-<pinref part="R5" gate="G$1" pin="2"/>
-<wire x1="33.02" y1="137.16" x2="35.56" y2="137.16" width="0.1524" layer="91"/>
-</segment>
-<segment>
-<pinref part="CAN(12V)" gate="G$1" pin="3"/>
-<wire x1="129.54" y1="104.14" x2="119.38" y2="104.14" width="0.1524" layer="91"/>
-<label x="119.38" y="104.14" size="1.27" layer="95"/>
-<pinref part="R7" gate="G$1" pin="2"/>
 </segment>
 <segment>
 <pinref part="R7" gate="G$1" pin="1"/>
-<wire x1="109.22" y1="104.14" x2="104.14" y2="104.14" width="0.1524" layer="91"/>
+<wire x1="119.38" y1="104.14" x2="104.14" y2="104.14" width="0.1524" layer="91"/>
+<label x="104.14" y="104.14" size="1.778" layer="95"/>
+</segment>
+<segment>
+<pinref part="R6" gate="G$1" pin="2"/>
+<wire x1="157.48" y1="104.14" x2="165.1" y2="104.14" width="0.1524" layer="91"/>
+<label x="157.48" y="104.14" size="1.778" layer="95"/>
 </segment>
 </net>
@@
 <net name="CLKOUT" class="0">
 <segment>
-<pinref part="CAN_IO" gate="1" pin="3"/>
-<wire x1="60.96" y1="152.4" x2="50.8" y2="152.4" width="0.1524" layer="91"/>
-<label x="50.8" y="152.4" size="1.778" layer="95"/>
-</segment>
-<segment>
 <pinref part="U$1" gate="G$1" pin="CLKOUT/SOF"/>
 <wire x1="43.18" y1="104.14" x2="35.56" y2="104.14" width="0.1524" layer="91"/>
@@
 <label x="35.56" y="101.6" size="1.524" layer="95"/>
 </segment>
-<segment>
-<wire x1="60.96" y1="149.86" x2="50.8" y2="149.86" width="0.1524" layer="91"/>
-<pinref part="CAN_IO" gate="1" pin="4"/>
-<label x="50.8" y="149.86" size="1.778" layer="95" font="fixed"/>
-</segment>
 </net>
 <net name="!TX1RTS" class="0">
@@
 <label x="35.56" y="99.06" size="1.524" layer="95"/>
 </segment>
-<segment>
-<pinref part="CAN_IO" gate="1" pin="5"/>
-<wire x1="60.96" y1="147.32" x2="50.8" y2="147.32" width="0.1524" layer="91"/>
-<label x="50.8" y="147.32" size="1.778" layer="95" font="fixed"/>
-</segment>
 </net>
 <net name="!TX2RTS" class="0">
@@
 <label x="35.56" y="93.98" size="1.524" layer="95" font="fixed"/>
 </segment>
-<segment>
-<pinref part="CAN_IO" gate="1" pin="6"/>
-<wire x1="60.96" y1="144.78" x2="50.8" y2="144.78" width="0.1524" layer="91"/>
-<label x="50.8" y="144.78" size="1.778" layer="95" font="fixed"/>
-</segment>
 </net>
 <net name="!CS" class="0">
@@
 </segment>
 </net>
+<net name="N$3" class="0">
+<segment>
+<pinref part="CAN(12V)" gate="G$1" pin="2"/>
+<pinref part="R8" gate="G$1" pin="2"/>
+<wire x1="121.92" y1="106.68" x2="129.54" y2="106.68" width="0.1524" layer="91"/>
+</segment>
+</net>
+<net name="N$4" class="0">
+<segment>
+<pinref part="CAN(12V)" gate="G$1" pin="3"/>
+<pinref part="R7" gate="G$1" pin="2"/>
+</segment>
+</net>
+<net name="N$11" class="0">
+<segment>
+<pinref part="CAN(12V)" gate="G$1" pin="5"/>
+<pinref part="R5" gate="G$1" pin="2"/>
+<wire x1="121.92" y1="99.06" x2="129.54" y2="99.06" width="0.1524" layer="91"/>
+</segment>
+</net>
+<net name="N$12" class="0">
+<segment>
+<pinref part="CAN(12V)" gate="G$1" pin="7"/>
+<pinref part="R6" gate="G$1" pin="1"/>
+<wire x1="147.32" y1="104.14" x2="144.78" y2="104.14" width="0.1524" layer="91"/>
+</segment>
+</net>

Commit message: Renamed some LEDs.  Closer to ordering GoodThopter12 boards.
git-svn-id: https://svn.code.sf.net/p/goodfet/code@1566 12e2690d-a6be-4b82-a7b7-67c4a43b65c8
Parts:
- renumbered RXLED to USBRX, RX_LED to CANRX, TXLED to USBTX, TX_LED to CANTX
Changed lines of the file:
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@@
 <part name="P+3" library="supply1" deviceset="VCC" device=""/>
 <part name="GND4" library="supply1" deviceset="GND" device=""/>
-<part name="RXLED" library="led" deviceset="LED" device="CHIP-LED0603"/>
-<part name="TXLED" library="led" deviceset="LED" device="CHIP-LED0603"/>
+<part name="USBRX" library="led" deviceset="LED" device="CHIP-LED0603"/>
+<part name="USBTX" library="led" deviceset="LED" device="CHIP-LED0603"/>
 <part name="P+4" library="supply1" deviceset="VCC" device=""/>
 <part name="R10" library="rcl" deviceset="R-US_" device="R0603" value="330"/>
@@
 <part name="C5" library="rcl" deviceset="C-EU" device="C0603" value="0.1uF"/>
 <part name="GND10" library="supply1" deviceset="GND" device=""/>
-<part name="TX_LED" library="led" deviceset="LED" device="CHIP-LED0603"/>
-<part name="RX_LED" library="led" deviceset="LED" device="CHIP-LED0603"/>
+<part name="CANTX" library="led" deviceset="LED" device="CHIP-LED0603"/>
+<part name="CANRX" library="led" deviceset="LED" device="CHIP-LED0603"/>
 <part name="R2" library="rcl" deviceset="R-US_" device="R0603" value="330"/>
 <part name="R3" library="rcl" deviceset="R-US_" device="R0603" value="330"/>
@@
 <instance part="P+3" gate="VCC" x="-15.24" y="55.88" rot="R90"/>
 <instance part="GND4" gate="1" x="-2.54" y="33.02"/>
-<instance part="RXLED" gate="G$1" x="38.1" y="38.1" rot="R270"/>
-<instance part="TXLED" gate="G$1" x="38.1" y="45.72" rot="R270"/>
+<instance part="USBRX" gate="G$1" x="38.1" y="38.1" rot="R270"/>
+<instance part="USBTX" gate="G$1" x="38.1" y="45.72" rot="R270"/>
 <instance part="P+4" gate="VCC" x="43.18" y="58.42"/>
 <instance part="R10" gate="G$1" x="43.18" y="50.8" rot="R90"/>
@@
 <instance part="C5" gate="G$1" x="-22.86" y="154.94" rot="R180"/>
 <instance part="GND10" gate="1" x="-22.86" y="149.86"/>
-<instance part="TX_LED" gate="G$1" x="30.48" y="114.3"/>
-<instance part="RX_LED" gate="G$1" x="22.86" y="114.3"/>
+<instance part="CANTX" gate="G$1" x="30.48" y="114.3"/>
+<instance part="CANRX" gate="G$1" x="22.86" y="114.3"/>
 <instance part="R2" gate="G$1" x="30.48" y="124.46" rot="R180"/>
 <instance part="R3" gate="G$1" x="43.18" y="121.92" rot="R180"/>
@@
 <wire x1="27.94" y1="38.1" x2="33.02" y2="38.1" width="0.1524" layer="91"/>
 <pinref part="IC2" gate="G$1" pin="RXLED"/>
-<pinref part="RXLED" gate="G$1" pin="C"/>
+<pinref part="USBRX" gate="G$1" pin="C"/>
 </segment>
 </net>
@@
 <wire x1="30.48" y1="45.72" x2="33.02" y2="45.72" width="0.1524" layer="91"/>
 <pinref part="IC2" gate="G$1" pin="TXLED"/>
-<pinref part="TXLED" gate="G$1" pin="C"/>
+<pinref part="USBTX" gate="G$1" pin="C"/>
 </segment>
 </net>
 <net name="N$8" class="0">
 <segment>
-<pinref part="TXLED" gate="G$1" pin="A"/>
+<pinref part="USBTX" gate="G$1" pin="A"/>
 <pinref part="R10" gate="G$1" pin="1"/>
 <wire x1="43.18" y1="45.72" x2="40.64" y2="45.72" width="0.1524" layer="91"/>
-<pinref part="RXLED" gate="G$1" pin="A"/>
+<pinref part="USBRX" gate="G$1" pin="A"/>
 <wire x1="40.64" y1="38.1" x2="43.18" y2="38.1" width="0.1524" layer="91"/>
 <wire x1="43.18" y1="38.1" x2="43.18" y2="45.72" width="0.1524" layer="91"/>
@@
 <wire x1="43.18" y1="109.22" x2="30.48" y2="109.22" width="0.1524" layer="91"/>
 <label x="35.56" y="109.22" size="1.778" layer="95"/>
-<pinref part="TX_LED" gate="G$1" pin="C"/>
+<pinref part="CANTX" gate="G$1" pin="C"/>
 </segment>
 <segment>
@@
 <wire x1="43.18" y1="106.68" x2="22.86" y2="106.68" width="0.1524" layer="91"/>
 <wire x1="22.86" y1="106.68" x2="22.86" y2="109.22" width="0.1524" layer="91"/>
-<pinref part="RX_LED" gate="G$1" pin="C"/>
+<pinref part="CANRX" gate="G$1" pin="C"/>
 </segment>
 <segment>
@@
 <net name="N$1" class="0">
 <segment>
-<pinref part="RX_LED" gate="G$1" pin="A"/>
+<pinref part="CANRX" gate="G$1" pin="A"/>
 <wire x1="22.86" y1="116.84" x2="22.86" y2="124.46" width="0.1524" layer="91"/>
 <wire x1="22.86" y1="124.46" x2="25.4" y2="124.46" width="0.1524" layer="91"/>
@@
 <net name="N$2" class="0">
 <segment>
-<pinref part="TX_LED" gate="G$1" pin="A"/>
+<pinref part="CANTX" gate="G$1" pin="A"/>
 <wire x1="30.48" y1="116.84" x2="30.48" y2="121.92" width="0.1524" layer="91"/>
 <wire x1="30.48" y1="121.92" x2="38.1" y2="121.92" width="0.1524" layer="91"/>

Commit message: Now the Sparkfun cable is default in the GoodThopter12. You can cut two traces and add two SMD resistors to use the older cable.
git-svn-id: https://svn.code.sf.net/p/goodfet/code@1567 12e2690d-a6be-4b82-a7b7-67c4a43b65c8
Parts:
- removed R5, R7: 0, rcl:R-US_R0603
Connections:
- removed net N$11: CAN(12V).5, R5.2
- removed net N$4: CAN(12V).3, R7.2
- net CANH: now also CAN(12V).3; no longer R7.1
- net CANL: now also CAN(12V).5; no longer R5.1
Other:
- note added: "Cut the traces for pins 3 and 5 if not using a Sparkfun cable."
- note added: "Do *NOT* populate R7 and R8 if using the Sparkfun cable."
- note added: "Pins 3,5 -- Sparkfun"
- note added: "Pins 7,2 -- ICS, GoodThopter11"
- note removed: "Populate *TWO* of R5, R6, R7, and R8 to choose your cable."
- note removed: "R5,R7 -- Pins 3,5 -- Sparkfun"
- note removed: "R6,R8 -- Pins 7,2 -- Intrepid Control Systems"
Changed lines of the file:
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@@
 <part name="Q2" library="crystal" deviceset="CRYSTAL" device="HC49UP" value="20MHz"/>
 <part name="U$2" library="MCP2551" deviceset="MCP2551" device=""/>
-<part name="R7" library="rcl" deviceset="R-US_" device="R0603" value="0"/>
 <part name="R8" library="rcl" deviceset="R-US_" device="R0603" value="0"/>
-<part name="R5" library="rcl" deviceset="R-US_" device="R0603" value="0"/>
 <part name="R6" library="rcl" deviceset="R-US_" device="R0603" value="0"/>
 </parts>
@@
 <text x="101.6" y="132.08" size="1.778" layer="104">PAY ATTENTION!</text>
 <text x="101.6" y="129.54" size="1.778" layer="104">Different CAN cables need different pins.</text>
-<text x="101.6" y="127" size="1.778" layer="104">Populate *TWO* of R5, R6, R7, and R8 to choose your cable.</text>
-<text x="101.6" y="124.46" size="1.778" layer="104">Known cables:</text>
-<text x="104.14" y="121.92" size="1.778" layer="104">R5,R7 -- Pins 3,5 -- Sparkfun</text>
-<text x="104.14" y="119.38" size="1.778" layer="104">R6,R8 -- Pins 7,2 -- Intrepid Control Systems</text>
+<text x="101.6" y="127" size="1.778" layer="104">Do *NOT* populate R7 and R8 if using the Sparkfun cable.</text>
+<text x="101.6" y="121.92" size="1.778" layer="104">Known cables:</text>
+<text x="104.14" y="119.38" size="1.778" layer="104">Pins 3,5 -- Sparkfun</text>
+<text x="104.14" y="116.84" size="1.778" layer="104">Pins 7,2 -- ICS, GoodThopter11</text>
+<text x="101.6" y="124.46" size="1.778" layer="104">Cut the traces for pins 3 and 5 if not using a Sparkfun cable.</text>
 </plain>
 <instances>
@@
 <instance part="Q2" gate="G$1" x="-22.86" y="104.14" rot="R90"/>
 <instance part="U$2" gate="G$1" x="-5.08" y="137.16"/>
-<instance part="R7" gate="G$1" x="124.46" y="104.14"/>
 <instance part="R8" gate="G$1" x="116.84" y="106.68"/>
-<instance part="R5" gate="G$1" x="116.84" y="99.06"/>
 <instance part="R6" gate="G$1" x="152.4" y="104.14"/>
 </instances>
@@
 </segment>
 <segment>
-<pinref part="R5" gate="G$1" pin="1"/>
-<wire x1="111.76" y1="99.06" x2="104.14" y2="99.06" width="0.1524" layer="91"/>
 <label x="104.14" y="99.06" size="1.778" layer="95"/>
+<pinref part="CAN(12V)" gate="G$1" pin="5"/>
+<wire x1="104.14" y1="99.06" x2="129.54" y2="99.06" width="0.1524" layer="91"/>
 </segment>
 </net>
@@
 </segment>
 <segment>
-<pinref part="R7" gate="G$1" pin="1"/>
-<wire x1="119.38" y1="104.14" x2="104.14" y2="104.14" width="0.1524" layer="91"/>
+<wire x1="129.54" y1="104.14" x2="104.14" y2="104.14" width="0.1524" layer="91"/>
 <label x="104.14" y="104.14" size="1.778" layer="95"/>
+<pinref part="CAN(12V)" gate="G$1" pin="3"/>
 </segment>
 <segment>
@@
 </segment>
 </net>
-<net name="N$4" class="0">
-<segment>
-<pinref part="CAN(12V)" gate="G$1" pin="3"/>
-<pinref part="R7" gate="G$1" pin="2"/>
-</segment>
-</net>
-<net name="N$11" class="0">
-<segment>
-<pinref part="CAN(12V)" gate="G$1" pin="5"/>
-<pinref part="R5" gate="G$1" pin="2"/>
-<wire x1="121.92" y1="99.06" x2="129.54" y2="99.06" width="0.1524" layer="91"/>
-</segment>
-</net>
