File: contrib/facedancer/raspdancer/pcb/raspdancer11_1.0.sch (EAGLE design)
At the start: 15 parts, among them Q1 12Mhz

Commit message: raspdancer pcb edited
thanks to Zac Franken for his tuning tips

git-svn-id: https://svn.code.sf.net/p/goodfet/code@1589 12e2690d-a6be-4b82-a7b7-67c4a43b65c8
Parts:
- removed C5: 1uF, 00_mylib:C1206
- J_RASP: device con-lsta:FE13-2 -> doegox:FE13-2
Connections:
- net GND: now also USB-MINIB.GND; no longer C5.1
- net VBUS: now also C1.2; no longer C5.2
- net VCC: no longer C1.2
Other:
- moved on the sheet: C1, JP3
Changed lines of the file:
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@@
 <part name="GND1" library="supply1" deviceset="GND" device=""/>
 <part name="GND2" library="supply1" deviceset="GND" device=""/>
-<part name="GND3" library="supply1" deviceset="GND" device=""/>
 <part name="GND4" library="supply1" deviceset="GND" device=""/>
 <part name="P+1" library="supply1" deviceset="VCC" device=""/>
-<part name="C1" library="00_mylib" deviceset="C" device="1206" value="1uF"/>
 <part name="C2" library="00_mylib" deviceset="C" device="1206" value="100nF"/>
 <part name="C3" library="00_mylib" deviceset="C" device="1206" value="18pF"/>
@@
 <part name="GND5" library="supply1" deviceset="GND" device=""/>
 <part name="GND8" library="supply1" deviceset="GND" device=""/>
-<part name="C5" library="00_mylib" deviceset="C" device="1206" value="1uF"/>
+<part name="C1" library="00_mylib" deviceset="C" device="1206" value="1uF"/>
 <part name="GND9" library="supply1" deviceset="GND" device=""/>
 <part name="R1" library="00_mylib" deviceset="R" device="1206" value="33"/>
 <part name="R2" library="00_mylib" deviceset="R" device="1206" value="33"/>
-<part name="J_RASP" library="con-lsta" deviceset="FE13-2" device=""/>
+<part name="J_RASP" library="doegox" deviceset="FE13-2" device=""/>
 <part name="P+2" library="supply1" deviceset="VCC" device=""/>
 <part name="GND10" library="supply1" deviceset="GND" device=""/>
@@
 <instance part="GND1" gate="1" x="92.71" y="80.01"/>
 <instance part="GND2" gate="1" x="74.93" y="80.01"/>
-<instance part="GND3" gate="1" x="39.37" y="83.82" rot="R270"/>
 <instance part="GND4" gate="1" x="66.04" y="99.06" rot="R180"/>
 <instance part="P+1" gate="VCC" x="59.69" y="90.17"/>
-<instance part="C1" gate="G$1" x="49.53" y="83.82" rot="R90"/>
 <instance part="C2" gate="G$1" x="66.04" y="88.9"/>
 <instance part="C3" gate="G$1" x="77.47" y="86.36"/>
 <instance part="C4" gate="G$1" x="90.17" y="86.36"/>
-<instance part="GND5" gate="1" x="-13.97" y="38.1"/>
+<instance part="GND5" gate="1" x="-13.97" y="35.56"/>
 <instance part="GND8" gate="1" x="58.42" y="27.94"/>
-<instance part="C5" gate="G$1" x="5.08" y="68.58"/>
+<instance part="C1" gate="G$1" x="5.08" y="68.58"/>
 <instance part="GND9" gate="1" x="5.08" y="80.01" rot="R180"/>
 <instance part="R1" gate="G$1" x="21.59" y="53.34"/>
@@
 <instance part="JP1" gate="A" x="132.08" y="50.8"/>
 <instance part="JP2" gate="A" x="104.14" y="81.28" rot="R90"/>
-<instance part="JP3" gate="G$1" x="-2.54" y="33.02" rot="R90"/>
+<instance part="JP3" gate="G$1" x="-2.54" y="30.48" rot="R90"/>
 <instance part="FRAME1" gate="G$1" x="-54.61" y="-36.83"/>
 <instance part="FRAME1" gate="G$2" x="92.71" y="-36.83"/>
@@
 <net name="GND" class="0">
 <segment>
-<wire x1="41.91" y1="83.82" x2="44.45" y2="83.82" width="0.1524" layer="91"/>
-<pinref part="GND3" gate="1" pin="GND"/>
-<pinref part="C1" gate="G$1" pin="1"/>
-</segment>
-<segment>
 <wire x1="66.04" y1="96.52" x2="66.04" y2="93.98" width="0.1524" layer="91"/>
 <pinref part="GND4" gate="1" pin="GND"/>
@@
 <pinref part="C3" gate="G$1" pin="2"/>
 <pinref part="GND2" gate="1" pin="GND"/>
-</segment>
-<segment>
-<wire x1="-13.97" y1="40.64" x2="-17.78" y2="40.64" width="0.1524" layer="91"/>
-<wire x1="0" y1="38.1" x2="0" y2="40.64" width="0.1524" layer="91"/>
-<wire x1="0" y1="40.64" x2="-13.97" y2="40.64" width="0.1524" layer="91"/>
-<junction x="-13.97" y="40.64"/>
-<pinref part="GND5" gate="1" pin="GND"/>
-<pinref part="JP3" gate="G$1" pin="1"/>
 </segment>
 <segment>
@@
 <segment>
 <wire x1="5.08" y1="77.47" x2="5.08" y2="73.66" width="0.1524" layer="91"/>
-<pinref part="C5" gate="G$1" pin="1"/>
+<pinref part="C1" gate="G$1" pin="1"/>
 <pinref part="GND9" gate="1" pin="GND"/>
 </segment>
@@
 <pinref part="GND11" gate="1" pin="GND"/>
 <wire x1="157.48" y1="72.39" x2="160.02" y2="72.39" width="0.1524" layer="91"/>
-<wire x1="160.02" y1="72.39" x2="165.1" y2="72.39" width="0.1524" layer="91"/>
 <wire x1="165.1" y1="72.39" x2="160.02" y2="72.39" width="0.1524" layer="91"/>
 <wire x1="160.02" y1="72.39" x2="160.02" y2="82.55" width="0.1524" layer="91"/>
@@
 <wire x1="160.02" y1="82.55" x2="157.48" y2="82.55" width="0.1524" layer="91"/>
 <junction x="160.02" y="72.39"/>
+<junction x="165.1" y="72.39"/>
 </segment>
 <segment>
@@
 <wire x1="134.62" y1="74.93" x2="134.62" y2="77.47" width="0.1524" layer="91"/>
 <wire x1="134.62" y1="77.47" x2="142.24" y2="77.47" width="0.1524" layer="91"/>
+</segment>
+<segment>
+<pinref part="USB-MINIB" gate="G$1" pin="GND"/>
+<pinref part="GND5" gate="1" pin="GND"/>
+<wire x1="-17.78" y1="40.64" x2="-13.97" y2="40.64" width="0.1524" layer="91"/>
+<wire x1="-13.97" y1="40.64" x2="-13.97" y2="38.1" width="0.1524" layer="91"/>
+<junction x="-13.97" y="40.64"/>
+<pinref part="JP3" gate="G$1" pin="1"/>
+<wire x1="-13.97" y1="40.64" x2="0" y2="40.64" width="0.1524" layer="91"/>
+<wire x1="0" y1="40.64" x2="0" y2="35.56" width="0.1524" layer="91"/>
 </segment>
 </net>
@@
 <wire x1="63.5" y1="83.82" x2="66.04" y2="83.82" width="0.1524" layer="91"/>
 <wire x1="66.04" y1="83.82" x2="66.04" y2="78.74" width="0.1524" layer="91"/>
-<wire x1="53.34" y1="83.82" x2="52.07" y2="83.82" width="0.1524" layer="91"/>
 <wire x1="66.04" y1="83.82" x2="66.04" y2="86.36" width="0.1524" layer="91"/>
 <wire x1="59.69" y1="87.63" x2="59.69" y2="83.82" width="0.1524" layer="91"/>
 <junction x="59.69" y="83.82"/>
-<junction x="53.34" y="83.82"/>
 <junction x="55.88" y="83.82"/>
 <junction x="63.5" y="83.82"/>
@@
 <pinref part="U1" gate="G$1" pin="VL@1"/>
 <pinref part="U1" gate="G$1" pin="VL@2"/>
-<pinref part="C1" gate="G$1" pin="2"/>
 <pinref part="C2" gate="G$1" pin="2"/>
 <pinref part="P+1" gate="VCC" pin="VCC"/>
@@
 <wire x1="-7.62" y1="50.8" x2="5.08" y2="50.8" width="0.1524" layer="91"/>
 <wire x1="5.08" y1="50.8" x2="5.08" y2="66.04" width="0.1524" layer="91"/>
-<wire x1="-7.62" y1="38.1" x2="-7.62" y2="50.8" width="0.1524" layer="91"/>
+<wire x1="-7.62" y1="35.56" x2="-7.62" y2="50.8" width="0.1524" layer="91"/>
 <wire x1="132.08" y1="43.18" x2="132.08" y2="24.13" width="0.1524" layer="91"/>
 <wire x1="132.08" y1="24.13" x2="5.08" y2="24.13" width="0.1524" layer="91"/>
@@
 <junction x="5.08" y="50.8"/>
 <pinref part="U1" gate="G$1" pin="VBCOMP"/>
-<pinref part="C5" gate="G$1" pin="2"/>
+<pinref part="C1" gate="G$1" pin="2"/>
 <pinref part="JP3" gate="G$1" pin="4"/>
 <pinref part="JP1" gate="A" pin="1"/>
@@
 <wire x1="-17.78" y1="48.26" x2="-2.54" y2="48.26" width="0.1524" layer="91"/>
 <wire x1="-2.54" y1="48.26" x2="13.97" y2="48.26" width="0.1524" layer="91"/>
-<wire x1="-2.54" y1="38.1" x2="-2.54" y2="48.26" width="0.1524" layer="91"/>
+<wire x1="-2.54" y1="35.56" x2="-2.54" y2="48.26" width="0.1524" layer="91"/>
 <junction x="-2.54" y="48.26"/>
 <pinref part="R1" gate="G$1" pin="1"/>
@@
 <wire x1="-17.78" y1="45.72" x2="-5.08" y2="45.72" width="0.1524" layer="91"/>
 <wire x1="-5.08" y1="45.72" x2="15.24" y2="45.72" width="0.1524" layer="91"/>
-<wire x1="-5.08" y1="38.1" x2="-5.08" y2="45.72" width="0.1524" layer="91"/>
+<wire x1="-5.08" y1="35.56" x2="-5.08" y2="45.72" width="0.1524" layer="91"/>
 <junction x="-5.08" y="45.72"/>
 <pinref part="R2" gate="G$1" pin="1"/>
